File: QtDash/Hardware/DashHat/dash-hat.sch (EAGLE design)
At the start: 123 parts, among them IC1 LM324, IC2 MCP3X083008, IC3 MCP23017SS, IC4 LM358D, IC5 IL300, IC6 LM358D, IC7 IL300, J1 CONN_20X2, J6 VOLVO_CONN_31, J7 VOLVO_CONN_32

Commit message: - added 2 more 5V sensor in channels (MAP and ambient temp) 	- started laying out sensor/ADC within limits of piHAT pcb section
Parts:
- removed D7, D8: BAT54, diode:BAT54
- added C15: 0.1uF, SparkFun-Capacitors:0.1UF-0603-25V-5%
- added C16: 1.0uF, SparkFun-Capacitors:1.0UF-0603-16V-10%
- added C17, C18: 10nF, SparkFun-Capacitors:10NF-0603-50V-10%
- added IC8: LM358D, digital_dash:LM358D
- added J10, J8: 455-1750-1-ND, SparkFun-Connectors:CONN_03
- added JP19, JP20: JUMPER-SMT_3_NO_SILK, SparkFun-Jumpers:JUMPER-SMT_3_NO_SILK
- added R63, R67: 1k, SparkFun-Resistors:1KOHM-0603-1/10W-1%
- added R64, R68: 330k, SparkFun-Resistors:330KOHM-0603-1/10W-1%
- added R65, R69: 100, SparkFun-Resistors:100OHM-0603-1/10W-1%
- added R66, R70: 640k, SparkFun-Resistors:390KOHM-0603-1/10W-1%
- D1, D2, D3, D4, D5, D6: value BAT54 -> BAT54S; device diode:BAT54 -> diode:BAT54S
Connections:
- net N$28 renamed OIL_PRESSURE
- net N$29 renamed OIL_TEMP
- removed net N$23: IC2.CH6
- removed net N$24: IC2.CH7
- new net ADC5_IN: C17.1, IC2.CH6, R64.1, R66.2
- new net ADC6_IN: C18.1, IC2.CH7, R68.1, R70.2
- new net AMBIENT_TEMP: JP20.3
- new net MAP_SENSOR: JP19.3
- new net N$19: JP18.2, R58.1
- new net N$28: IC8A.-IN, IC8A.OUT, R64.2
- new net N$29: D5.C1A2, IC8A.+IN, R65.2
- new net N$35: IC8B.-IN, IC8B.OUT, R68.2
- new net N$36: D6.C1A2, IC8B.+IN, R69.2
- new net N$37: JP20.2, R67.1, R69.1
- new net SENSOR5_IN: J10.2, JP19.1
- new net SENSOR6_IN: J8.2, JP20.1
- net 5V: now also C15.1, C16.1, D1.C2, D2.C2, D3.C2, D4.C2, D5.C2, D6.C2, IC8A.V+, J10.3, J8.3, R63.2, R67.2; no longer D1.C, D3.C, D5.C, D7.C
- net GND: now also C15.2, C16.2, C17.2, C18.2, D1.A1, D2.A1, D3.A1, D4.A1, D5.A1, D6.A1, IC8A.V-, J10.1, J8.1, R66.1, R70.1; no longer D2.A, D4.A, D6.A, D8.A
- net N$11: now also D3.C1A2; no longer D5.A, D6.C
- net N$15: now also D4.C1A2; no longer D7.A, D8.C
- net N$3: now also D1.C1A2; no longer D1.A, D2.C
- net N$34: now also JP19.2, R63.1, R65.1; no longer JP18.1
- net N$7: now also D2.C1A2; no longer D3.A, D4.C
- net SIG_12V_IN2: now also JP18.1; no longer JP18.2, R58.1
Other:
- moved on the sheet: C1, C2, C3, C4, C5, C6, IC1A, IC1B, IC1C, IC1D, J2, J3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
