File: QtDash/Hardware/DashHat/dash-hat.sch (EAGLE design)
At the start: 160 parts, among them IC1 LMV614, IC10 MAX9924, IC11 ZXTR2105FQ, IC2 MCP3X083008, IC3 MCP23017SS, IC4 LM358D, IC5 IL300, IC6 TSV912D, IC7 IL300, IC8 TSV912D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

Commit message: topic/hardware-revc: 	- Analog input layout with new connector is done -- need to check on connector footprint as there is a dimension error 	- TODO: replace switched 12V power and GND with molex connector (right angle?)
Parts:
- added JP15: VSS- Jumper, SparkFun-Jumpers:JUMPER-SMT_2_NO_SILK
Connections:
- net N$48 renamed VSS+
- removed net N$49: J11.VSS-, R7.1
- new net VSS-: J11.VSS-, JP15.1, R7.1
- net 5V: now also J27.S; no longer J21.S
- net GND-ISO: now also JP15.2
- net SENSOR4_IN: now also J21.S; no longer J25.S
- net SENSOR5_IN: now also J25.S; no longer J26.S
- net SENSOR6_IN: now also J26.S; no longer J27.S
Other:
- moved on the sheet: J21, J22, J23, J24, J25, J26, J27, J28
Changed lines of the file:
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@@
 <part name="GND52" library="SparkFun-PowerSymbols" deviceset="GND" device=""/>
 <part name="J2" library="digital_dash" deviceset="CONN_04X2" device=""/>
+<part name="JP15" library="SparkFun-Jumpers" deviceset="JUMPER-SMT_2_NO" device="_SILK" value="VSS- Jumper"/>
+<part name="GND-ISO30" library="SparkFun-PowerSymbols" deviceset="GND-ISO" device=""/>
 </parts>
 <sheets>
@@
 <instance part="SUPPLY61" gate="G$1" x="506.73" y="237.49"/>
 <instance part="GND45" gate="1" x="494.03" y="198.12" rot="MR0"/>
-<instance part="SUPPLY52" gate="G$1" x="271.78" y="416.56"/>
-<instance part="GND52" gate="1" x="271.78" y="391.16"/>
-<instance part="J2" gate="1" x="279.4" y="414.02"/>
-<instance part="J2" gate="2" x="279.4" y="411.48"/>
-<instance part="J2" gate="3" x="279.4" y="408.94"/>
-<instance part="J2" gate="4" x="279.4" y="406.4"/>
-<instance part="J2" gate="5" x="279.4" y="403.86"/>
-<instance part="J2" gate="6" x="279.4" y="401.32"/>
-<instance part="J2" gate="7" x="279.4" y="398.78"/>
-<instance part="J2" gate="8" x="279.4" y="396.24"/>
+<instance part="SUPPLY52" gate="G$1" x="40.64" y="401.32"/>
+<instance part="GND52" gate="1" x="58.42" y="388.62"/>
+<instance part="J2" gate="1" x="66.04" y="411.48"/>
+<instance part="J2" gate="2" x="66.04" y="408.94"/>
+<instance part="J2" gate="3" x="66.04" y="406.4"/>
+<instance part="J2" gate="4" x="66.04" y="403.86"/>
+<instance part="J2" gate="5" x="66.04" y="401.32"/>
+<instance part="J2" gate="6" x="66.04" y="398.78"/>
+<instance part="J2" gate="7" x="66.04" y="396.24"/>
+<instance part="J2" gate="8" x="66.04" y="393.7"/>
+<instance part="JP15" gate="G$1" x="403.86" y="274.32" rot="R270"/>
+<instance part="GND-ISO30" gate="G$1" x="403.86" y="266.7"/>
 </instances>
 <busses>
@@
 <segment>
 <pinref part="J2" gate="4" pin="S"/>
-<wire x1="276.86" y1="406.4" x2="271.78" y2="406.4" width="0.1524" layer="91"/>
-<label x="271.78" y="406.4" size="1.27" layer="95" rot="R180" xref="yes"/>
+<wire x1="63.5" y1="403.86" x2="58.42" y2="403.86" width="0.1524" layer="91"/>
+<label x="58.42" y="403.86" size="1.27" layer="95" rot="R180" xref="yes"/>
 </segment>
 </net>
@@
 <segment>
 <pinref part="J2" gate="3" pin="S"/>
-<wire x1="276.86" y1="408.94" x2="271.78" y2="408.94" width="0.1524" layer="91"/>
-<label x="271.78" y="408.94" size="1.27" layer="95" rot="R180" xref="yes"/>
+<wire x1="63.5" y1="406.4" x2="58.42" y2="406.4" width="0.1524" layer="91"/>
+<label x="58.42" y="406.4" size="1.27" layer="95" rot="R180" xref="yes"/>
 </segment>
 </net>
@@
 <segment>
 <pinref part="J2" gate="2" pin="S"/>
-<wire x1="276.86" y1="411.48" x2="271.78" y2="411.48" width="0.1524" layer="91"/>
-<label x="271.78" y="411.48" size="1.27" layer="95" rot="R180" xref="yes"/>
+<wire x1="63.5" y1="408.94" x2="58.42" y2="408.94" width="0.1524" layer="91"/>
+<label x="58.42" y="408.94" size="1.27" layer="95" rot="R180" xref="yes"/>
 </segment>
 </net>
@@
 </segment>
 <segment>
-<wire x1="276.86" y1="403.86" x2="271.78" y2="403.86" width="0.1524" layer="91"/>
-<label x="271.78" y="403.86" size="1.27" layer="95" rot="R180" xref="yes"/>
-<pinref part="J2" gate="5" pin="S"/>
+<pinref part="J2" gate="1" pin="S"/>
+<wire x1="63.5" y1="411.48" x2="58.42" y2="411.48" width="0.1524" layer="91"/>
+<label x="58.42" y="411.48" size="1.27" layer="95" rot="R180" xref="yes"/>
 </segment>
 </net>
@@
 </segment>
 <segment>
-<wire x1="276.86" y1="396.24" x2="271.78" y2="396.24" width="0.1524" layer="91"/>
-<wire x1="271.78" y1="396.24" x2="271.78" y2="393.7" width="0.1524" layer="91"/>
+<wire x1="63.5" y1="393.7" x2="58.42" y2="393.7" width="0.1524" layer="91"/>
+<wire x1="58.42" y1="393.7" x2="58.42" y2="391.16" width="0.1524" layer="91"/>
 <pinref part="GND52" gate="1" pin="GND"/>
 <pinref part="J2" gate="8" pin="S"/>
@@
 <segment>
 <pinref part="SUPPLY52" gate="G$1" pin="5V"/>
-<wire x1="276.86" y1="414.02" x2="271.78" y2="414.02" width="0.1524" layer="91"/>
-<wire x1="271.78" y1="414.02" x2="271.78" y2="416.56" width="0.1524" layer="91"/>
-<pinref part="J2" gate="1" pin="S"/>
+<wire x1="40.64" y1="396.24" x2="40.64" y2="401.32" width="0.1524" layer="91"/>
+<pinref part="J2" gate="7" pin="S"/>
+<wire x1="63.5" y1="396.24" x2="40.64" y2="396.24" width="0.1524" layer="91"/>
 </segment>
 </net>
@@
 <pinref part="GND-ISO29" gate="G$1" pin="GND-ISO"/>
 </segment>
+<segment>
+<pinref part="JP15" gate="G$1" pin="2"/>
+<pinref part="GND-ISO30" gate="G$1" pin="GND-ISO"/>
+</segment>
 </net>
 <net name="BRAKE_FAILURE_N" class="0">
@@
 </segment>
 <segment>
-<wire x1="276.86" y1="401.32" x2="271.78" y2="401.32" width="0.1524" layer="91"/>
-<label x="271.78" y="401.32" size="1.27" layer="95" rot="R180" xref="yes"/>
-<pinref part="J2" gate="6" pin="S"/>
+<pinref part="J2" gate="5" pin="S"/>
+<wire x1="63.5" y1="401.32" x2="58.42" y2="401.32" width="0.1524" layer="91"/>
+<label x="58.42" y="401.32" size="1.27" layer="95" rot="R180" xref="yes"/>
 </segment>
 </net>
@@
 </segment>
 <segment>
-<wire x1="276.86" y1="398.78" x2="271.78" y2="398.78" width="0.1524" layer="91"/>
-<label x="271.78" y="398.78" size="1.27" layer="95" rot="R180" xref="yes"/>
-<pinref part="J2" gate="7" pin="S"/>
+<pinref part="J2" gate="6" pin="S"/>
+<wire x1="63.5" y1="398.78" x2="58.42" y2="398.78" width="0.1524" layer="91"/>
+<label x="58.42" y="398.78" size="1.27" layer="95" rot="R180" xref="yes"/>
 </segment>
 </net>
@@
 </segment>
 </net>
-<net name="N$48" class="0">
+<net name="VSS+" class="0">
 <segment>
 <pinref part="J11" gate="G$1" pin="VSS+"/>
@@
 <wire x1="386.08" y1="241.3" x2="388.62" y2="241.3" width="0.1524" layer="91"/>
 <wire x1="388.62" y1="241.3" x2="397.51" y2="250.19" width="0.1524" layer="91"/>
+<label x="388.62" y="241.3" size="1.27" layer="95" rot="R270" xref="yes"/>
 </segment>
 </net>
-<net name="N$49" class="0">
+<net name="VSS-" class="0">
 <segment>
 <pinref part="J11" gate="G$1" pin="VSS-"/>
@@
 <pinref part="R7" gate="G$1" pin="1"/>
 <wire x1="388.62" y1="248.92" x2="397.51" y2="240.03" width="0.1524" layer="91"/>
+<label x="388.62" y="248.92" size="1.27" layer="95" rot="R90" xref="yes"/>
+</segment>
+<segment>
+<pinref part="JP15" gate="G$1" pin="1"/>
+<wire x1="403.86" y1="279.4" x2="403.86" y2="281.94" width="0.1524" layer="91"/>
+<label x="403.86" y="281.94" size="1.27" layer="95" rot="R180" xref="yes"/>
 </segment>
 </net>

Commit message: topic/hardware-revc: 	- added right angle nano-fit molex connector for switched 12V power 	- added 4 user inputs on the remaining 4 pins of MCP23017 	- added pwm output on pin 18 with 3.3V pullup 	- added user inputs to dash_lights.h -- likely need to pull this out and/or rework
Parts:
- removed J18, J19, J9: (no value), SparkFun-Connectors:CONN_02PTH4
- added J3: CONN_04RIGHT-ANGLE, digital_dash:CONN_04RIGHT-ANGLE
- added J4: CONN_04, digital_dash:CONN_04
- added J5: PWM_OUT, SparkFun-Connectors:CONN_03
- added R60: 20k, digital_dash:RC0603JR-0720KL
- added R64, R66, R68, R70: 1k, digital_dash:RC0603JR-071KL
Connections:
- new net GPIO18: J1.12, J5.2, R60.1
- new net USER_IN1: IC3.GPB4, J41.S, R64.2
- new net USER_IN2: IC3.GPB5, J42.S, R66.2
- new net USER_IN3: IC3.GPB6, J43.S, R68.2
- new net USER_IN4: IC3.GPB7, J44.S, R70.2
- net 12V: now also J31.S, J32.S; no longer J18.1, J18.2, J9.1, J9.2
- net 3.3V: now also R60.2, R64.1, R66.1, R68.1, R70.1
- net 5V: now also J5.3; no longer J19.2
- net GND: now also J5.1; no longer J19.1
- net GND-ISO: now also J33.S, J34.S

Commit message: topic/hardware-revc: 	- reduced pullups directly on GPIOs from 1k to 20k 	- added pwm to rpi4 config and initial_turbo 	- slight layout changes
Parts:
- R16, R54, R76: value 1k -> 20k; device digital_dash:RC0603JR-071KL -> digital_dash:RC0603JR-0720KL
Changed lines of the file:
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@@
 <setting verticaltext="up"/>
 </settings>
-<grid distance="0.05" unitdist="inch" unit="inch" style="lines" multiple="1" display="no" altdistance="0.01" altunitdist="inch" altunit="inch"/>
+<grid distance="0.1" unitdist="inch" unit="inch" style="lines" multiple="1" display="no" altdistance="0.01" altunitdist="inch" altunit="inch"/>
 <layers>
 <layer number="1" name="Top" color="4" fill="1" visible="no" active="no"/>
@@
 <part name="SUPPLY55" library="SparkFun-PowerSymbols" deviceset="3.3V" device=""/>
 <part name="GND50" library="SparkFun-PowerSymbols" deviceset="GND" device=""/>
-<part name="R76" library="digital_dash" deviceset="RC0603JR" device="" technology="-071KL" value="1k"/>
+<part name="R76" library="digital_dash" deviceset="RC0603JR" device="" technology="-0720KL" value="20k"/>
 <part name="R82" library="digital_dash" deviceset="RES_D+" device=""/>
 <part name="J20" library="SparkFun-Connectors" deviceset="CONN_02" device="PTH4"/>
@@
 <part name="SUPPLY60" library="SparkFun-PowerSymbols" deviceset="12V" device=""/>
 <part name="R15" library="digital_dash" deviceset="RC0603JR" device="" technology="-071KL" value="1k"/>
-<part name="R16" library="digital_dash" deviceset="RC0603JR" device="" technology="-071KL" value="1k"/>
-<part name="R54" library="digital_dash" deviceset="RC0603JR" device="" technology="-071KL" value="1k"/>
+<part name="R16" library="digital_dash" deviceset="RC0603JR" device="" technology="-0720KL" value="20k"/>
+<part name="R54" library="digital_dash" deviceset="RC0603JR" device="" technology="-0720KL" value="20k"/>
 <part name="SUPPLY61" library="SparkFun-PowerSymbols" deviceset="3.3V" device=""/>
 <part name="GND45" library="SparkFun-PowerSymbols" deviceset="GND" device=""/>

Commit message: topic/hardware-revc: 	- added MCP2515 and SN65HVD230 to board 	- didn't use split termination or common mode choke for CAN -- if there is EMI issues that'll be one (of likely many) place to look
Parts:
- added C30, C31: 100n, digital_dash:CL10B104MB8NNNC
- added C32, C33: 22p, digital_dash:CL10C220JB81PNC
- added D9: PESD1CAN, diode:PESD1CAN
- added IC12: SN65HVD230D, digital_dash:SN65HVD230D
- added J8: (no value), digital_dash:CONN_02
- added JP16: SPI_CS_SEL, SparkFun-Jumpers:JUMPER-SMT_3_NO_SILK
- added R77: 120 1%, digital_dash:RC0603FR-07120RL
- added R80: 1k, digital_dash:RC0603JR-071KL
- added R81: 20k, digital_dash:RC0603JR-0720KL
- added U1: MCP2515, SparkFun-IC-Comms:MCP2515(MCP2510)SO
- added X1: 12MHz, digital_dash:ECS-120-20-3X-TR
Connections:
- new net !CAN_SPI_CS: JP16.2, U1>NAME.CS
- new net CANH: D9.1, IC12.CANH, J8.1, R77.2
- new net CANL: D9.2, IC12.CANL, J8.2, R77.1
- new net GPIO25: J1.22, U1>NAME.INT
- new net N$12: IC12.S, R80.1
- new net N$18: C32.2, U1>NAME.OSC1, X1.1
- new net N$31: C33.1, U1>NAME.OSC2, X1.2
- new net N$37: IC12.RXD, U1>NAME.RXCAN
- new net N$40: IC12.TXD, U1>NAME.TXCAN
- new net N$43: R81.1, U1>NAME.RESET
- net 3.3V: now also C30.1, C31.1, IC12.VCC, R81.2, U1P.VDD
- net GND: now also C30.2, C31.2, C32.1, C33.2, D9.3, IC12.GND, R80.2, U1P.VSS
- net SPI_CE0_N: now also JP16.3
- net SPI_CE1_N: now also JP16.1
- net SPI_CLK: now also U1>NAME.SCK
- net SPI_MISO: now also U1>NAME.SO
- net SPI_MOSI: now also U1>NAME.SI
Other:
- moved on the sheet: C23, C24, C25, C26, C27, C28, IC10, IC11, J11, J20, J21, J31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

Commit message: topic/hardware-revc: 	- added parts list for rev c
Other:
- note added: "CAN Transceiver"
Changed lines of the file:
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@@
 <setting verticaltext="up"/>
 </settings>
-<grid distance="0.05" unitdist="inch" unit="inch" style="lines" multiple="1" display="no" altdistance="0.01" altunitdist="inch" altunit="inch"/>
+<grid distance="0.1" unitdist="inch" unit="inch" style="lines" multiple="1" display="no" altdistance="0.01" altunitdist="inch" altunit="inch"/>
 <layers>
 <layer number="1" name="Top" color="4" fill="1" visible="no" active="no"/>
@@
 </attributes>
 <variantdefs>
+<variantdef name="REVC" current="yes"/>
 </variantdefs>
 <classes>
@@
 <part name="OK1" library="digital_dash" deviceset="ILQ1" device="X009"/>
 <part name="R17" library="digital_dash" deviceset="RC0603JR" device="" technology="-07470RL" value="470R"/>
-<part name="R18" library="digital_dash" deviceset="RC0603JR" device="" technology="-07470RL" value="470R"/>
+<part name="R18" library="digital_dash" deviceset="RC0603JR" device="" technology="-07470RL" value="470R">
+<variant name="REVC" populate="no"/>
+</part>
 <part name="SUPPLY13" library="SparkFun-PowerSymbols" deviceset="12V" device=""/>
 <part name="R19" library="digital_dash" deviceset="RC0603JR" device="" technology="-07470RL" value="470R"/>
 <part name="GND24" library="SparkFun-PowerSymbols" deviceset="GND" device=""/>
 <part name="SUPPLY14" library="SparkFun-PowerSymbols" deviceset="3.3V" device=""/>
-<part name="R20" library="digital_dash" deviceset="RC0603JR" device="" technology="-07470RL" value="470R"/>
+<part name="R20" library="digital_dash" deviceset="RC0603JR" device="" technology="-07470RL" value="470R">
+<variant name="REVC" populate="no"/>
+</part>
 <part name="R21" library="digital_dash" deviceset="RC0603JR" device="" technology="-07470RL" value="470R"/>
 <part name="SUPPLY15" library="SparkFun-PowerSymbols" deviceset="12V" device=""/>
@@
 <part name="SUPPLY16" library="SparkFun-PowerSymbols" deviceset="3.3V" device=""/>
 <part name="GND26" library="SparkFun-PowerSymbols" deviceset="GND" device=""/>
-<part name="R23" library="digital_dash" deviceset="RC0603JR" device="" technology="-07470RL" value="470R"/>
+<part name="R23" library="digital_dash" deviceset="RC0603JR" device="" technology="-07470RL" value="470R">
+<variant name="REVC" populate="no"/>
+</part>
 <part name="R24" library="digital_dash" deviceset="RC0603JR" device="" technology="-07470RL" value="470R"/>
 <part name="SUPPLY17" library="SparkFun-PowerSymbols" deviceset="12V" device=""/>
 <part name="R25" library="digital_dash" deviceset="RC0603JR" device="" technology="-07470RL" value="470R"/>
-<part name="R26" library="digital_dash" deviceset="RC0603JR" device="" technology="-07470RL" value="470R"/>
+<part name="R26" library="digital_dash" deviceset="RC0603JR" device="" technology="-07470RL" value="470R">
+<variant name="REVC" populate="no"/>
+</part>
 <part name="SUPPLY18" library="SparkFun-PowerSymbols" deviceset="12V" device=""/>
 <part name="R27" library="digital_dash" deviceset="RC0603JR" device="" technology="-07470RL" value="470R"/>
@@
 <part name="OK2" library="digital_dash" deviceset="ILQ1" device="X009"/>
 <part name="R29" library="digital_dash" deviceset="RC0603JR" device="" technology="-07470RL" value="470R"/>
-<part name="R30" library="digital_dash" deviceset="RC0603JR" device="" technology="-07470RL" value="470R"/>
+<part name="R30" library="digital_dash" deviceset="RC0603JR" device="" technology="-07470RL" value="470R">
+<variant name="REVC" populate="no"/>
+</part>
 <part name="SUPPLY21" library="SparkFun-PowerSymbols" deviceset="12V" device=""/>
 <part name="R31" library="digital_dash" deviceset="RC0603JR" device="" technology="-07470RL" value="470R"/>
@@
 <part name="SUPPLY22" library="SparkFun-PowerSymbols" deviceset="3.3V" device=""/>
 <part name="R32" library="digital_dash" deviceset="RC0603JR" device="" technology="-07470RL" value="470R"/>
-<part name="R33" library="digital_dash" deviceset="RC0603JR" device="" technology="-07470RL" value="470R"/>
+<part name="R33" library="digital_dash" deviceset="RC0603JR" device="" technology="-07470RL" value="470R">
+<variant name="REVC" populate="no"/>
+</part>
 <part name="SUPPLY23" library="SparkFun-PowerSymbols" deviceset="12V" device=""/>
 <part name="R34" library="digital_dash" deviceset="RC0603JR" device="" technology="-07470RL" value="470R"/>
 <part name="SUPPLY24" library="SparkFun-PowerSymbols" deviceset="3.3V" device=""/>
 <part name="GND34" library="SparkFun-PowerSymbols" deviceset="GND" device=""/>
-<part name="R35" library="digital_dash" deviceset="RC0603JR" device="" technology="-07470RL" value="470R"/>
+<part name="R35" library="digital_dash" deviceset="RC0603JR" device="" technology="-07470RL" value="470R">
+<variant name="REVC" populate="no"/>
+</part>
 <part name="R36" library="digital_dash" deviceset="RC0603JR" device="" technology="-07470RL" value="470R"/>
 <part name="SUPPLY25" library="SparkFun-PowerSymbols" deviceset="12V" device=""/>
-<part name="R37" library="digital_dash" deviceset="RC0603JR" device="" technology="-07470RL" value="470R"/>
+<part name="R37" library="digital_dash" deviceset="RC0603JR" device="" technology="-07470RL" value="470R">
+<variant name="REVC" populate="no"/>
+</part>
 <part name="R38" library="digital_dash" deviceset="RC0603JR" device="" technology="-07470RL" value="470R"/>
 <part name="SUPPLY26" library="SparkFun-PowerSymbols" deviceset="12V" device=""/>
@@
 <part name="C10" library="digital_dash" deviceset="CL" device="" technology="10A105KA8NNNC" value="1u"/>
 <part name="OK3" library="digital_dash" deviceset="ILQ1" device="X009"/>
-<part name="R41" library="digital_dash" deviceset="RC0603JR" device="" technology="-07470RL" value="470R"/>
-<part name="R42" library="digital_dash" deviceset="RC0603JR" device="" technology="-07470RL" value="470R"/>
+<part name="R41" library="digital_dash" deviceset="RC0603JR" device="" technology="-07470RL" value="470R">
+<variant name="REVC" populate="no"/>
+</part>
+<part name="R42" library="digital_dash" deviceset="RC0603JR" device="" technology="-07470RL" value="470R">
+<variant name="REVC" populate="no"/>
+</part>
 <part name="SUPPLY30" library="SparkFun-PowerSymbols" deviceset="12V" device=""/>
 <part name="R43" library="digital_dash" deviceset="RC0603JR" device="" technology="-07470RL" value="470R"/>
@@
 <part name="SUPPLY31" library="SparkFun-PowerSymbols" deviceset="3.3V" device=""/>
 <part name="R44" library="digital_dash" deviceset="RC0603JR" device="" technology="-07470RL" value="470R"/>
-<part name="R45" library="digital_dash" deviceset="RC0603JR" device="" technology="-07470RL" value="470R"/>
+<part name="R45" library="digital_dash" deviceset="RC0603JR" device="" technology="-07470RL" value="470R">
+<variant name="REVC" populate="no"/>
+</part>
 <part name="SUPPLY32" library="SparkFun-PowerSymbols" deviceset="12V" device=""/>
 <part name="R46" library="digital_dash" deviceset="RC0603JR" device="" technology="-07470RL" value="470R"/>
@@
 <part name="GND44" library="SparkFun-PowerSymbols" deviceset="GND" device=""/>
 <part name="R47" library="digital_dash" deviceset="RC0603JR" device="" technology="-07470RL" value="470R"/>
-<part name="R48" library="digital_dash" deviceset="RC0603JR" device="" technology="-07470RL" value="470R"/>
+<part name="R48" library="digital_dash" deviceset="RC0603JR" device="" technology="-07470RL" value="470R">
+<variant name="REVC" populate="no"/>
+</part>
 <part name="SUPPLY34" library="SparkFun-PowerSymbols" deviceset="12V" device=""/>
-<part name="R49" library="digital_dash" deviceset="RC0603JR" device="" technology="-07470RL" value="470R"/>
-<part name="R50" library="digital_dash" deviceset="RC0603JR" device="" technology="-07470RL" value="470R"/>
+<part name="R49" library="digital_dash" deviceset="RC0603JR" device="" technology="-07470RL" value="470R">
+<variant name="REVC" populate="no"/>
+</part>
+<part name="R50" library="digital_dash" deviceset="RC0603JR" device="" technology="-07470RL" value="470R">
+<variant name="REVC" populate="no"/>
+</part>
 <part name="SUPPLY35" library="SparkFun-PowerSymbols" deviceset="12V" device=""/>
 <part name="R51" library="digital_dash" deviceset="RC0603JR" device="" technology="-07470RL" value="470R"/>
@@
 <text x="110.49" y="417.83" size="5.08" layer="97">Switched 12V</text>
 <text x="412.75" y="245.11" size="5.08" layer="97">VSS Input Coniditioning</text>
+<text x="387.35" y="349.25" size="5.08" layer="97">CAN Transceiver</text>
 </plain>
 <instances>
