File: QtDash/Hardware/DashHat/dash-hat.sch (EAGLE design)
At the start: 179 parts, among them IC1 LMV614, IC10 MAX9924, IC11 ZXTR2105FQ, IC12 SN65HVD230D, IC2 MCP3X083008, IC3 MCP23017SS, IC4 LM358D, IC5 IL300, IC6 TSV912D, IC7 IL300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

Commit message: topic/hardware-revc: 	- fixed (hopefully) some string comparision issues in sensor utils and config 	- updated mcp2515 and transceiver circuit -- todo: check dimensions of cheap amazon JST style plug
Parts:
- renumbered U1 to IC13
Changed lines of the file:
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@@
 </attributes>
 <variantdefs>
-<variantdef name="REVC" current="yes"/>
+<variantdef name="REVC"/>
 </variantdefs>
 <classes>
@@
 <part name="R70" library="digital_dash" deviceset="RC0603JR" device="" technology="-071KL" value="1k"/>
 <part name="SUPPLY56" library="SparkFun-PowerSymbols" deviceset="3.3V" device=""/>
-<part name="U1" library="SparkFun-IC-Comms" deviceset="MCP2515(MCP2510)" device="SO" value="MCP2515"/>
+<part name="IC13" library="SparkFun-IC-Comms" deviceset="MCP2515(MCP2510)" device="SO" value="MCP2515"/>
 <part name="D9" library="diode" deviceset="PESD1CAN" device=""/>
 <part name="IC12" library="digital_dash" deviceset="SN65HVD23" device="" technology="0D"/>
@@
 <instance part="R70" gate="G$1" x="491.49" y="74.93" rot="R90"/>
 <instance part="SUPPLY56" gate="G$1" x="469.9" y="71.12"/>
-<instance part="U1" gate="&gt;NAME" x="431.8" y="322.58"/>
+<instance part="IC13" gate="&gt;NAME" x="431.8" y="322.58"/>
 <instance part="D9" gate="G$1" x="508" y="307.34" rot="R270"/>
 <instance part="IC12" gate="G$1" x="485.14" y="325.12"/>
@@
 <instance part="R81" gate="G$1" x="406.4" y="312.42" rot="R180"/>
 <instance part="SUPPLY63" gate="G$1" x="391.16" y="314.96"/>
-<instance part="U1" gate="P" x="441.96" y="279.4"/>
+<instance part="IC13" gate="P" x="441.96" y="279.4"/>
 <instance part="SUPPLY64" gate="G$1" x="441.96" y="289.56"/>
 <instance part="GND51" gate="1" x="441.96" y="266.7" rot="MR0"/>
@@
 </segment>
 <segment>
-<pinref part="U1" gate="P" pin="VSS"/>
+<pinref part="IC13" gate="P" pin="VSS"/>
 <pinref part="GND51" gate="1" pin="GND"/>
 <wire x1="441.96" y1="271.78" x2="441.96" y2="269.24" width="0.1524" layer="91"/>
@@
 </segment>
 <segment>
-<pinref part="U1" gate="P" pin="VDD"/>
+<pinref part="IC13" gate="P" pin="VDD"/>
 <pinref part="SUPPLY64" gate="G$1" pin="3.3V"/>
 <wire x1="441.96" y1="287.02" x2="441.96" y2="289.56" width="0.1524" layer="91"/>
@@
 </segment>
 <segment>
-<pinref part="U1" gate="&gt;NAME" pin="SI"/>
+<pinref part="IC13" gate="&gt;NAME" pin="SI"/>
 <wire x1="416.56" y1="320.04" x2="408.94" y2="320.04" width="0.1524" layer="91"/>
 <label x="408.94" y="320.04" size="1.27" layer="95" rot="R180" xref="yes"/>
@@
 </segment>
 <segment>
-<pinref part="U1" gate="&gt;NAME" pin="SO"/>
+<pinref part="IC13" gate="&gt;NAME" pin="SO"/>
 <wire x1="416.56" y1="317.5" x2="408.94" y2="317.5" width="0.1524" layer="91"/>
 <label x="408.94" y="317.5" size="1.27" layer="95" rot="R180" xref="yes"/>
@@
 </segment>
 <segment>
-<pinref part="U1" gate="&gt;NAME" pin="SCK"/>
+<pinref part="IC13" gate="&gt;NAME" pin="SCK"/>
 <wire x1="416.56" y1="322.58" x2="408.94" y2="322.58" width="0.1524" layer="91"/>
 <label x="408.94" y="322.58" size="1.27" layer="95" rot="R180" xref="yes"/>
@@
 <pinref part="IC12" gate="G$1" pin="RXD"/>
 <wire x1="469.9" y1="317.5" x2="459.74" y2="317.5" width="0.1524" layer="91"/>
-<pinref part="U1" gate="&gt;NAME" pin="RXCAN"/>
+<pinref part="IC13" gate="&gt;NAME" pin="RXCAN"/>
 <wire x1="459.74" y1="317.5" x2="449.58" y2="327.66" width="0.1524" layer="91"/>
 </segment>
@@
 <pinref part="IC12" gate="G$1" pin="TXD"/>
 <wire x1="469.9" y1="332.74" x2="459.74" y2="332.74" width="0.1524" layer="91"/>
-<pinref part="U1" gate="&gt;NAME" pin="TXCAN"/>
+<pinref part="IC13" gate="&gt;NAME" pin="TXCAN"/>
 <wire x1="459.74" y1="332.74" x2="449.58" y2="322.58" width="0.1524" layer="91"/>
 </segment>
@@
 <net name="N$43" class="0">
 <segment>
-<pinref part="U1" gate="&gt;NAME" pin="RESET"/>
+<pinref part="IC13" gate="&gt;NAME" pin="RESET"/>
 <pinref part="R81" gate="G$1" pin="1"/>
 <wire x1="416.56" y1="312.42" x2="411.48" y2="312.42" width="0.1524" layer="91"/>
@@
 </segment>
 <segment>
-<pinref part="U1" gate="&gt;NAME" pin="CS"/>
+<pinref part="IC13" gate="&gt;NAME" pin="CS"/>
 <wire x1="416.56" y1="325.12" x2="408.94" y2="325.12" width="0.1524" layer="91"/>
 <label x="408.94" y="325.12" size="1.27" layer="95" rot="R180" xref="yes"/>
@@
 <net name="N$18" class="0">
 <segment>
-<pinref part="U1" gate="&gt;NAME" pin="OSC1"/>
+<pinref part="IC13" gate="&gt;NAME" pin="OSC1"/>
 <wire x1="416.56" y1="335.28" x2="393.7" y2="335.28" width="0.1524" layer="91"/>
 <wire x1="393.7" y1="335.28" x2="393.7" y2="340.36" width="0.1524" layer="91"/>
@@
 <net name="N$31" class="0">
 <segment>
-<pinref part="U1" gate="&gt;NAME" pin="OSC2"/>
+<pinref part="IC13" gate="&gt;NAME" pin="OSC2"/>
 <wire x1="416.56" y1="332.74" x2="393.7" y2="332.74" width="0.1524" layer="91"/>
 <wire x1="393.7" y1="332.74" x2="393.7" y2="325.12" width="0.1524" layer="91"/>
@@
 </segment>
 <segment>
-<pinref part="U1" gate="&gt;NAME" pin="INT"/>
+<pinref part="IC13" gate="&gt;NAME" pin="INT"/>
 <wire x1="449.58" y1="312.42" x2="452.12" y2="312.42" width="0.1524" layer="91"/>
 <label x="452.12" y="312.42" size="1.27" layer="95" xref="yes"/>
