File: QtDash/Hardware/DashHat/Board Revisions/Rev A/dash-hat.brd (EAGLE design)
At the start: 107.8 x 66.8 mm, 163 parts, among them IC1 LM324, IC2 MCP3X083008, IC3 MCP23017SS, IC4 LM358D, IC5 IL300, IC6 LM358D, IC7 IL300, IC8 LM358D, IC9 DS1374, J1 CONN_20X2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

Commit message: - update Board Revisions/Rev A schematic with final assembly values notes on final assembly
Parts:
- R10: value 1k -> 91
- R11: value 1k -> 43
- R12: value 1k -> 150
- R67: value 1k -> 6.49k
- R9: value 1k -> 470R
Changed lines of the file:
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@@
 </attributes>
 <variantdefs>
+<variantdef name="Rev A Final Assembly" current="yes"/>
 </variantdefs>
 <classes>
@@
 <element name="C5" library="digital_dash" package="0603" value="100n" x="22.86" y="22.86" rot="MR180"/>
 <element name="J2" library="SparkFun-Connectors" package="1X02" value="" x="11.43" y="2.032"/>
-<element name="R9" library="digital_dash" package="0603" value="1k" x="11.698" y="9.418" rot="R90"/>
+<element name="R9" library="digital_dash" package="0603" value="470R" x="11.698" y="9.418" rot="R90"/>
 <element name="J3" library="SparkFun-Connectors" package="1X02" value="" x="17.018" y="2.032"/>
-<element name="R10" library="digital_dash" package="0603" value="1k" x="17.272" y="9.398" rot="R90"/>
+<element name="R10" library="digital_dash" package="0603" value="91" x="17.272" y="9.398" rot="R90"/>
 <element name="J4" library="SparkFun-Connectors" package="1X02" value="" x="22.606" y="2.032"/>
-<element name="R11" library="digital_dash" package="0603" value="1k" x="22.86" y="9.398" rot="R90"/>
+<element name="R11" library="digital_dash" package="0603" value="43" x="22.86" y="9.398" rot="R90"/>
 <element name="J5" library="SparkFun-Connectors" package="1X02" value="" x="28.194" y="2.032"/>
-<element name="R12" library="digital_dash" package="0603" value="1k" x="28.448" y="9.398" rot="R90"/>
+<element name="R12" library="digital_dash" package="0603" value="150" x="28.448" y="9.398" rot="R90"/>
 <element name="R1" library="digital_dash" package="0603" value="100R" x="13.236" y="9.378" rot="R90"/>
 <element name="R3" library="digital_dash" package="0603" value="330k" x="18.542" y="18.542" rot="R90"/>
@@
 <element name="OK1" library="digital_dash" package="SMD16" value="ILQ1X009" x="62.484" y="47.498" rot="R180"/>
 <element name="R17" library="digital_dash" package="0603" value="470R" x="70.866" y="38.354"/>
-<element name="R18" library="digital_dash" package="0603" value="470R" x="70.866" y="41.402" rot="R180"/>
+<element name="R18" library="digital_dash" package="0603" value="470R" x="70.866" y="41.402" populate="no" rot="R180"/>
 <element name="R19" library="digital_dash" package="0603" value="470R" x="55.118" y="39.878" rot="R270"/>
-<element name="R20" library="digital_dash" package="0603" value="470R" x="70.866" y="46.482"/>
+<element name="R20" library="digital_dash" package="0603" value="470R" x="70.866" y="46.482" populate="no"/>
 <element name="R21" library="digital_dash" package="0603" value="470R" x="70.866" y="42.926" rot="R180"/>
 <element name="R22" library="digital_dash" package="0603" value="470R" x="55.118" y="44.45" rot="R90"/>
-<element name="R23" library="digital_dash" package="0603" value="470R" x="70.866" y="48.006"/>
+<element name="R23" library="digital_dash" package="0603" value="470R" x="70.866" y="48.006" populate="no"/>
 <element name="R24" library="digital_dash" package="0603" value="470R" x="70.866" y="51.562" rot="R180"/>
 <element name="R25" library="digital_dash" package="0603" value="470R" x="70.866" y="56.134"/>
-<element name="R26" library="digital_dash" package="0603" value="470R" x="70.866" y="53.086" rot="R180"/>
+<element name="R26" library="digital_dash" package="0603" value="470R" x="70.866" y="53.086" populate="no" rot="R180"/>
 <element name="R27" library="digital_dash" package="0603" value="470R" x="55.118" y="50.038" rot="R270"/>
 <element name="R28" library="digital_dash" package="0603" value="470R" x="55.118" y="54.864" rot="R90"/>
 <element name="OK2" library="digital_dash" package="SMD16" value="ILQ1X009" x="62.484" y="47.498" rot="MR0"/>
 <element name="R29" library="digital_dash" package="0603" value="470R" x="70.612" y="56.134" rot="MR180"/>
-<element name="R30" library="digital_dash" package="0603" value="470R" x="70.612" y="53.34" rot="MR0"/>
+<element name="R30" library="digital_dash" package="0603" value="470R" x="70.612" y="53.34" populate="no" rot="MR0"/>
 <element name="R31" library="digital_dash" package="0603" value="470R" x="55.118" y="54.864" rot="MR90"/>
 <element name="R32" library="digital_dash" package="0603" value="470R" x="70.612" y="48.006" rot="MR180"/>
-<element name="R33" library="digital_dash" package="0603" value="470R" x="70.612" y="51.816" rot="MR0"/>
+<element name="R33" library="digital_dash" package="0603" value="470R" x="70.612" y="51.816" populate="no" rot="MR0"/>
 <element name="R34" library="digital_dash" package="0603" value="470R" x="55.118" y="50.038" rot="MR270"/>
-<element name="R35" library="digital_dash" package="0603" value="470R" x="70.612" y="46.482" rot="MR180"/>
+<element name="R35" library="digital_dash" package="0603" value="470R" x="70.612" y="46.482" populate="no" rot="MR180"/>
 <element name="R36" library="digital_dash" package="0603" value="470R" x="70.612" y="42.926" rot="MR0"/>
-<element name="R37" library="digital_dash" package="0603" value="470R" x="70.612" y="38.354" rot="MR180"/>
+<element name="R37" library="digital_dash" package="0603" value="470R" x="70.612" y="38.354" populate="no" rot="MR180"/>
 <element name="R38" library="digital_dash" package="0603" value="470R" x="70.612" y="41.402" rot="MR0"/>
 <element name="R39" library="digital_dash" package="0603" value="470R" x="55.118" y="44.45" rot="MR90"/>
@@
 <element name="R43" library="digital_dash" package="0603" value="470R" x="55.118" y="14.986" rot="R270"/>
 <element name="R44" library="digital_dash" package="0603" value="470R" x="71.628" y="21.59"/>
-<element name="R45" library="digital_dash" package="0603" value="470R" x="71.628" y="18.034" rot="R180"/>
+<element name="R45" library="digital_dash" package="0603" value="470R" x="71.628" y="18.034" populate="no" rot="R180"/>
 <element name="R46" library="digital_dash" package="0603" value="470R" x="55.118" y="19.558" rot="R90"/>
 <element name="R47" library="digital_dash" package="0603" value="470R" x="71.628" y="23.114"/>
-<element name="R48" library="digital_dash" package="0603" value="470R" x="71.628" y="26.67" rot="R180"/>
+<element name="R48" library="digital_dash" package="0603" value="470R" x="71.628" y="26.67" populate="no" rot="R180"/>
 <element name="R49" library="digital_dash" package="0603" value="470R" x="71.628" y="31.242"/>
 <element name="R50" library="digital_dash" package="0603" value="470R" x="71.628" y="28.194" rot="R180"/>
@@
 <element name="C15" library="digital_dash" package="0603" value="100n" x="38.608" y="21.844" rot="R180"/>
 <element name="C16" library="digital_dash" package="0603" value="1u" x="38.608" y="23.368" rot="R180"/>
-<element name="R63" library="digital_dash" package="0603" value="1k" x="34.036" y="9.652" rot="R90"/>
+<element name="R63" library="digital_dash" package="0603" value="1k" x="34.036" y="9.652" populate="no" rot="R90"/>
 <element name="R64" library="digital_dash" package="0603" value="330k" x="32.766" y="18.542"/>
 <element name="C17" library="digital_dash" package="0603" value="10n" x="32.766" y="15.494"/>
@@
 <element name="R66" library="digital_dash" package="0603" value="620k" x="32.766" y="17.018" rot="R180"/>
 <element name="JP19" library="SparkFun-Jumpers" package="SMT-JUMPER_3_NO_SILK" value="JUMPER-SMT_3_NO_SILK" x="35.56" y="6.604" rot="R180"/>
-<element name="R67" library="digital_dash" package="0603" value="1k" x="43.688" y="9.652" rot="R90"/>
+<element name="R67" library="digital_dash" package="0603" value="6.49k" x="43.688" y="9.652" rot="R90"/>
 <element name="R68" library="digital_dash" package="0603" value="330k" x="43.434" y="18.288" rot="R270"/>
 <element name="C18" library="digital_dash" package="0603" value="10n" x="46.482" y="18.288" rot="R270"/>
@@
 <element name="C20" library="digital_dash" package="0603" value="1u" x="32.258" y="46.482"/>
 <element name="R75" library="digital_dash" package="0603" value="1k" x="32.258" y="44.704" rot="R180"/>
-<element name="S1" library="SparkFun-Switches" package="TACTILE_SWITCH_SMD_6.0X3.5MM" value="RST_SW" x="24.384" y="50.546" rot="R270">
+<element name="S1" library="SparkFun-Switches" package="TACTILE_SWITCH_SMD_6.0X3.5MM" value="RST_SW" x="24.384" y="50.546" populate="no" rot="R270">
 <attribute name="PROD_ID" value="SWCH-14278" x="24.384" y="50.546" size="1.778" layer="27" rot="R270" display="off"/>
 <attribute name="SF_SKU" value="COM-08229" x="24.384" y="50.546" size="1.778" layer="27" rot="R270" display="off"/>
@@
 <element name="JP24" library="SparkFun-Jumpers" package="SMT-JUMPER_3_NO_SILK" value="TACH_INPUT_SEL" x="9.398" y="47.752" rot="R90"/>
 <element name="R76" library="digital_dash" package="0603" value="1k" x="20.066" y="59.69" rot="R180"/>
-<element name="R77" library="digital_dash" package="0603" value="1k" x="25.146" y="59.69" rot="R180"/>
+<element name="R77" library="digital_dash" package="0603" value="1k" x="25.146" y="59.69" populate="no" rot="R180"/>
 <element name="R78" library="digital_dash" package="0603" value="1k" x="9.652" y="59.69" rot="R180"/>
-<element name="R79" library="digital_dash" package="0603" value="1k" x="14.732" y="59.69" rot="R180"/>
+<element name="R79" library="digital_dash" package="0603" value="1k" x="14.732" y="59.69" populate="no" rot="R180"/>
 <element name="R82" library="resistor" package="0617/17" value="" x="95.758" y="62.992" rot="R180"/>
 </elements>
