File: QtDash/Hardware/DashHat/Board Revisions/Rev A/dash-hat.sch (EAGLE design)
At the start: 163 parts, among them IC1 LM324, IC2 MCP3X083008, IC3 MCP23017SS, IC4 LM358D, IC5 IL300, IC6 LM358D, IC7 IL300, IC8 LM358D, IC9 DS1374, J1 CONN_20X2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

Commit message: - update Board Revisions/Rev A schematic with final assembly values notes on final assembly
Parts:
- R10: value 1k -> 91
- R11: value 1k -> 43
- R12: value 1k -> 150
- R67: value 1k -> 6.49k
- R9: value 1k -> 470R; device digital_dash:RC0603JR-071KL -> digital_dash:RC0603JR-07470RL
Other:
- note added: "Jumper to GPIO19"
- note added: "Jumper to GPIO6"
- note added: "Sandwich 100nF capacitor on R56 and R62. This should stop oscillations on the outputs."
- note added: "Used a 68R 5W."
- moved on the sheet: BT1
