File: QtDash/Hardware/VSS Adapter/vss_adapter.sch (EAGLE design)
At the start: 21 parts, among them IC1 MAX9924, IC2 ZXTR2105FQ, J1 VOLVO_CONN_VSS, Q1 310mA/60V/1.6Ω

Commit message: bugfix/hardware-revA-issues: 	- added jumper from VSS- to ground just in case and up-reved VSS input board 	-
Parts:
- added JP2: VSS-_GND, SparkFun-Jumpers:JUMPER-SMT_2_NO_SILK
Connections:
- net N$1 renamed VSS+
- net N$3 renamed IN+
- net N$4 renamed IN-
- net N$7 renamed VSS2_OUT
- removed net N$2: J1.VSS-, R2.1
- new net VSS-: J1.VSS-, JP2.2, R2.1
- net GND: now also JP2.1
Other:
- moved on the sheet: C1, C2, C3, C4, C5, C6, IC1, IC2, J1, J2, J3, J4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
