File: QtDash/Hardware/Cold Start Power Supply/Dash Power Supply/dash_power_supply.sch (EAGLE design)
At the start: 55 parts, among them IC1 LM5060, IC2 LM3488, Q1 IPB042N10N3GATMA1, Q2 IPB042N10N3GATMA1, Q3 BC816-25HVL, Q4 BSC027N04LSG

Commit message: topic/component-optimization: 	- udpated supply and input protection board
Parts:
- R10: value 20k -> 20R; device SparkFun-Resistors:20KOHM-0603-1/10W-5% -> digital_dash:RC0603JR-0720RL
Connections:
- net VBATT: now also Q1.D; no longer Q2.D
- net VIN: now also Q2.D; no longer Q1.D
Other:
- moved on the sheet: Q1, Q2
