File: QtDash/Hardware/Cold Start Power Supply/Dash Power Supply - Kicad/cold-start-power-supply/cold-start-power-supply.kicad_sch (KiCad schematic)
At the start: 29 parts, among them IC1 LM3488, J1 Conn_01x02, J2 Conn_01x02, Q1 BSC026N08NS5

Commit message: 82-bom-missing: 	- updated Kicad cold start power supply schematic with part numbers and generated BOM
Parts:
- C1, C2: PN (none) -> EEE-FK1K3R3R
- C9: PN CL32A107MPVNNNE -> CL32A107MPVNNNE
- Q1: value BSC026N08NS5 -> DMTH6002LPS-13
